Commit message: Update

File: src/robot_custom_description/models/robot_01/model_backup copy.urdf (robot description, URDF)
Before this commit: robot robot_01, 48 links, 47 joints
Joints:
- joint robot_01/marker_joint: limit lower=0 upper=0 effort=0 velocity=0 -> (none); type prismatic -> fixed

File: src/robot_custom_description/models/robot_02/model.urdf (robot description, URDF)
Before this commit: robot robot_02, 48 links, 47 joints
Links:
- removed link robot_02/marker_link
- added link marker_id_02, mass 0.0144; collision mesh filename=package://robot_custom_description/models/robot_02/meshes/m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; visual mesh filename=package://robot_custom_description/models/markers/marker_02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
Joints:
- joint robot_02/marker_joint: child robot_02/marker_link -> marker_id_02
