Commit message: Both robots working on rviz2

File: src/robot_custom_description/models/robot_01/model copy.urdf (robot description, URDF)
Before this commit: robot robot_02, 48 links, 47 joints
Links:
- removed link marker_id_02
- removed link robot_02/b1_link
- removed link robot_02/b2_link
- removed link robot_02/b3_link
- removed link robot_02/base_link
- removed link robot_02/gr_ref_link
- removed link robot_02/m1_link
- removed link robot_02/m1_r1_link
- removed link robot_02/m1_r2_link
- removed link robot_02/m1_r3_link
- removed link robot_02/m1_r4_link
- removed link robot_02/m1_r5_link
- removed link robot_02/m1_r6_link
- removed link robot_02/m1_r7_link
- removed link robot_02/m1_r8_link
- removed link robot_02/m1_r9_link
- removed link robot_02/m2_link
- removed link robot_02/m2_r1_link
- removed link robot_02/m2_r2_link
- removed link robot_02/m2_r3_link
- removed link robot_02/m2_r4_link
- removed link robot_02/m2_r5_link
- removed link robot_02/m2_r6_link
- removed link robot_02/m2_r7_link
- removed link robot_02/m2_r8_link
- removed link robot_02/m2_r9_link
- removed link robot_02/m3_link
- removed link robot_02/m3_r1_link
- removed link robot_02/m3_r2_link
- removed link robot_02/m3_r3_link
- removed link robot_02/m3_r4_link
- removed link robot_02/m3_r5_link
- removed link robot_02/m3_r6_link
- removed link robot_02/m3_r7_link
- removed link robot_02/m3_r8_link
- removed link robot_02/m3_r9_link
- removed link robot_02/m4_link
- removed link robot_02/m4_r1_link
- removed link robot_02/m4_r2_link
- removed link robot_02/m4_r3_link
- removed link robot_02/m4_r4_link
- removed link robot_02/m4_r5_link
- removed link robot_02/m4_r6_link
- removed link robot_02/m4_r7_link
- removed link robot_02/m4_r8_link
- removed link robot_02/m4_r9_link
- removed link robot_02/p1_link
- removed link robot_02/p2_link
- added link marker_id_01, mass 0.0144; collision mesh filename=package://robot_custom_description/models/robot_01/meshes/m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; visual mesh filename=package://robot_custom_description/models/markers/marker_01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
- added link robot_01/b1_link, mass 0.233473387976464; collision mesh filename=package://robot_custom_description/models/robot_01/meshes/b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; visual mesh filename=package://robot_custom_description/models/robot_01/meshes/b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
- added link robot_01/b2_link, mass 0.21624485416319; collision mesh filename=package://robot_custom_description/models/robot_01/meshes/b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; visual mesh filename=package://robot_custom_description/models/robot_01/meshes/b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
- added link robot_01/b3_link, mass 0.194452851189113; collision mesh filename=package://robot_custom_description/models/robot_01/meshes/b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; visual mesh filename=package://robot_custom_description/models/robot_01/meshes/b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
- added link robot_01/base_link, mass 1.30966382009507; collision mesh filename=package://robot_custom_description/models/robot_01/meshes/b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; visual mesh filename=package://robot_custom_description/models/robot_01/meshes/b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
- added link robot_01/gr_ref_link, mass 0.0005; collision mesh filename=package://robot_custom_description/models/robot_01/meshes/g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; visual mesh filename=package://robot_custom_description/models/robot_01/meshes/g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
- added link robot_01/m1_link, mass 0.348747920870875; collision mesh filename=package://robot_custom_description/models/robot_01/meshes/m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; visual mesh filename=package://robot_custom_description/models/robot_01/meshes/m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
- added link robot_01/m1_r1_link, mass 0.00929201442640384; collision mesh filename=package://robot_custom_description/models/robot_01/meshes/m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; visual mesh filename=package://robot_custom_description/models/robot_01/meshes/m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
- added link robot_01/m1_r2_link, mass 0.00929201442640375; collision mesh filename=package://robot_custom_description/models/robot_01/meshes/m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; visual mesh filename=package://robot_custom_description/models/robot_01/meshes/m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
- added link robot_01/m1_r3_link, mass 0.00929201442640375; collision mesh filename=package://robot_custom_description/models/robot_01/meshes/m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; visual mesh filename=package://robot_custom_description/models/robot_01/meshes/m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
- added link robot_01/m1_r4_link, mass 0.00929201442640384; collision mesh filename=package://robot_custom_description/models/robot_01/meshes/m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; visual mesh filename=package://robot_custom_description/models/robot_01/meshes/m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
- added link robot_01/m1_r5_link, mass 0.00929201442640384; collision mesh filename=package://robot_custom_description/models/robot_01/meshes/m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; visual mesh filename=package://robot_custom_description/models/robot_01/meshes/m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
- added link robot_01/m1_r6_link, mass 0.00929201442640384; collision mesh filename=package://robot_custom_description/models/robot_01/meshes/m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; visual mesh filename=package://robot_custom_description/models/robot_01/meshes/m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
- added link robot_01/m1_r7_link, mass 0.0092920144264038; collision mesh filename=package://robot_custom_description/models/robot_01/meshes/m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; visual mesh filename=package://robot_custom_description/models/robot_01/meshes/m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
- added link robot_01/m1_r8_link, mass 0.00929201442640389; collision mesh filename=package://robot_custom_description/models/robot_01/meshes/m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; visual mesh filename=package://robot_custom_description/models/robot_01/meshes/m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
- added link robot_01/m1_r9_link, mass 0.00929201442640389; collision mesh filename=package://robot_custom_description/models/robot_01/meshes/m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; visual mesh filename=package://robot_custom_description/models/robot_01/meshes/m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
- added link robot_01/m2_link, mass 0.33159524637187; collision mesh filename=package://robot_custom_description/models/robot_01/meshes/m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; visual mesh filename=package://robot_custom_description/models/robot_01/meshes/m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
- added link robot_01/m2_r1_link, mass 0.00929201442640389; collision mesh filename=package://robot_custom_description/models/robot_01/meshes/m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; visual mesh filename=package://robot_custom_description/models/robot_01/meshes/m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
- added link robot_01/m2_r2_link, mass 0.00929201442640389; collision mesh filename=package://robot_custom_description/models/robot_01/meshes/m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; visual mesh filename=package://robot_custom_description/models/robot_01/meshes/m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
- added link robot_01/m2_r3_link, mass 0.00929201442640374; collision mesh filename=package://robot_custom_description/models/robot_01/meshes/m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; visual mesh filename=package://robot_custom_description/models/robot_01/meshes/m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
- added link robot_01/m2_r4_link, mass 0.00929201442640389; collision mesh filename=package://robot_custom_description/models/robot_01/meshes/m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; visual mesh filename=package://robot_custom_description/models/robot_01/meshes/m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
- added link robot_01/m2_r5_link, mass 0.00929201442640384; collision mesh filename=package://robot_custom_description/models/robot_01/meshes/m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; visual mesh filename=package://robot_custom_description/models/robot_01/meshes/m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
- added link robot_01/m2_r6_link, mass 0.00929201442640375; collision mesh filename=package://robot_custom_description/models/robot_01/meshes/m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; visual mesh filename=package://robot_custom_description/models/robot_01/meshes/m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
- added link robot_01/m2_r7_link, mass 0.00929201442640375; collision mesh filename=package://robot_custom_description/models/robot_01/meshes/m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; visual mesh filename=package://robot_custom_description/models/robot_01/meshes/m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
- added link robot_01/m2_r8_link, mass 0.00929201442640375; collision mesh filename=package://robot_custom_description/models/robot_01/meshes/m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; visual mesh filename=package://robot_custom_description/models/robot_01/meshes/m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
- added link robot_01/m2_r9_link, mass 0.00929201442640389; collision mesh filename=package://robot_custom_description/models/robot_01/meshes/m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; visual mesh filename=package://robot_custom_description/models/robot_01/meshes/m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
- added link robot_01/m3_link, mass 0.331595246320107; collision mesh filename=package://robot_custom_description/models/robot_01/meshes/m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; visual mesh filename=package://robot_custom_description/models/robot_01/meshes/m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
- added link robot_01/m3_r1_link, mass 0.00929201442640375; collision mesh filename=package://robot_custom_description/models/robot_01/meshes/m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; visual mesh filename=package://robot_custom_description/models/robot_01/meshes/m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
- added link robot_01/m3_r2_link, mass 0.00929201442640389; collision mesh filename=package://robot_custom_description/models/robot_01/meshes/m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; visual mesh filename=package://robot_custom_description/models/robot_01/meshes/m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
- added link robot_01/m3_r3_link, mass 0.00929201442640384; collision mesh filename=package://robot_custom_description/models/robot_01/meshes/m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; visual mesh filename=package://robot_custom_description/models/robot_01/meshes/m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
- added link robot_01/m3_r4_link, mass 0.00929201442640389; collision mesh filename=package://robot_custom_description/models/robot_01/meshes/m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; visual mesh filename=package://robot_custom_description/models/robot_01/meshes/m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
- added link robot_01/m3_r5_link, mass 0.00929201442640375; collision mesh filename=package://robot_custom_description/models/robot_01/meshes/m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; visual mesh filename=package://robot_custom_description/models/robot_01/meshes/m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
- added link robot_01/m3_r6_link, mass 0.00929201442640375; collision mesh filename=package://robot_custom_description/models/robot_01/meshes/m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; visual mesh filename=package://robot_custom_description/models/robot_01/meshes/m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
- added link robot_01/m3_r7_link, mass 0.00929201442640389; collision mesh filename=package://robot_custom_description/models/robot_01/meshes/m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; visual mesh filename=package://robot_custom_description/models/robot_01/meshes/m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
- added link robot_01/m3_r8_link, mass 0.00929201442640384; collision mesh filename=package://robot_custom_description/models/robot_01/meshes/m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; visual mesh filename=package://robot_custom_description/models/robot_01/meshes/m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
- added link robot_01/m3_r9_link, mass 0.00929201442640384; collision mesh filename=package://robot_custom_description/models/robot_01/meshes/m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; visual mesh filename=package://robot_custom_description/models/robot_01/meshes/m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
- added link robot_01/m4_link, mass 0.348747920793599; collision mesh filename=package://robot_custom_description/models/robot_01/meshes/m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; visual mesh filename=package://robot_custom_description/models/robot_01/meshes/m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
- added link robot_01/m4_r1_link, mass 0.00929201442640389; collision mesh filename=package://robot_custom_description/models/robot_01/meshes/m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; visual mesh filename=package://robot_custom_description/models/robot_01/meshes/m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
- added link robot_01/m4_r2_link, mass 0.00929201442640379; collision mesh filename=package://robot_custom_description/models/robot_01/meshes/m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; visual mesh filename=package://robot_custom_description/models/robot_01/meshes/m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
- added link robot_01/m4_r3_link, mass 0.00929201442640384; collision mesh filename=package://robot_custom_description/models/robot_01/meshes/m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; visual mesh filename=package://robot_custom_description/models/robot_01/meshes/m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
- added link robot_01/m4_r4_link, mass 0.00929201442640389; collision mesh filename=package://robot_custom_description/models/robot_01/meshes/m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; visual mesh filename=package://robot_custom_description/models/robot_01/meshes/m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
- added link robot_01/m4_r5_link, mass 0.00929201442640384; collision mesh filename=package://robot_custom_description/models/robot_01/meshes/m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; visual mesh filename=package://robot_custom_description/models/robot_01/meshes/m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
- added link robot_01/m4_r6_link, mass 0.00929201442640389; collision mesh filename=package://robot_custom_description/models/robot_01/meshes/m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; visual mesh filename=package://robot_custom_description/models/robot_01/meshes/m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
- added link robot_01/m4_r7_link, mass 0.00929201442640375; collision mesh filename=package://robot_custom_description/models/robot_01/meshes/m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; visual mesh filename=package://robot_custom_description/models/robot_01/meshes/m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
- added link robot_01/m4_r8_link, mass 0.00929201442640389; collision mesh filename=package://robot_custom_description/models/robot_01/meshes/m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; visual mesh filename=package://robot_custom_description/models/robot_01/meshes/m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
- added link robot_01/m4_r9_link, mass 0.00929201442640389; collision mesh filename=package://robot_custom_description/models/robot_01/meshes/m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; visual mesh filename=package://robot_custom_description/models/robot_01/meshes/m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
- added link robot_01/p1_link, mass 0.0032658; collision mesh filename=package://robot_custom_description/models/robot_01/meshes/p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; visual mesh filename=package://robot_custom_description/models/robot_01/meshes/p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
- added link robot_01/p2_link, mass 0.0032658; collision mesh filename=package://robot_custom_description/models/robot_01/meshes/p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; visual mesh filename=package://robot_custom_description/models/robot_01/meshes/p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
Joints:
- removed joint robot_02/b1_joint
- removed joint robot_02/b2_joint
- removed joint robot_02/b3_joint
- removed joint robot_02/base_joint
- removed joint robot_02/gr_ref_joint
- removed joint robot_02/m1_joint
- removed joint robot_02/m1_r1_joint
- removed joint robot_02/m1_r2_joint
- removed joint robot_02/m1_r3_joint
- removed joint robot_02/m1_r4_joint
- removed joint robot_02/m1_r5_joint
- removed joint robot_02/m1_r6_joint
- removed joint robot_02/m1_r7_joint
- removed joint robot_02/m1_r8_joint
- removed joint robot_02/m1_r9_joint
- removed joint robot_02/m2_joint
- removed joint robot_02/m2_r1_joint
- removed joint robot_02/m2_r2_joint
- removed joint robot_02/m2_r3_joint
- removed joint robot_02/m2_r4_joint
- removed joint robot_02/m2_r5_joint
- removed joint robot_02/m2_r6_joint
- removed joint robot_02/m2_r7_joint
- removed joint robot_02/m2_r8_joint
- removed joint robot_02/m2_r9_joint
- removed joint robot_02/m3_joint
- removed joint robot_02/m3_r1_joint
- removed joint robot_02/m3_r2_joint
- removed joint robot_02/m3_r3_joint
- removed joint robot_02/m3_r4_joint
- removed joint robot_02/m3_r5_joint
- removed joint robot_02/m3_r6_joint
- removed joint robot_02/m3_r7_joint
- removed joint robot_02/m3_r8_joint
- removed joint robot_02/m3_r9_joint
- removed joint robot_02/m4_joint
- removed joint robot_02/m4_r1_joint
- removed joint robot_02/m4_r2_joint
- removed joint robot_02/m4_r3_joint
- removed joint robot_02/m4_r4_joint
- removed joint robot_02/m4_r5_joint
- removed joint robot_02/m4_r6_joint
- removed joint robot_02/m4_r7_joint
- removed joint robot_02/m4_r8_joint
- removed joint robot_02/m4_r9_joint
- removed joint robot_02/p1_joint
- removed joint robot_02/p2_joint
- added joint robot_01/b1_joint: type revolute, parent robot_01/base_link, child robot_01/b1_link, origin xyz=0.0749999999999994 0 0.0620000000000007 rpy=-1.5707963267949 0 0, axis 0 0 1, limit lower=0 upper=0 effort=0 velocity=0
- added joint robot_01/b2_joint: type revolute, parent robot_01/b1_link, child robot_01/b2_link, origin xyz=0 -0.075 0 rpy=0 0 0, axis 0 0 1, limit lower=0 upper=0 effort=0 velocity=0
- added joint robot_01/b3_joint: type revolute, parent robot_01/b2_link, child robot_01/b3_link, origin xyz=0 -0.0699999999999995 0 rpy=0 0 0, axis 0 0 1, limit lower=0 upper=0 effort=0 velocity=0
- added joint robot_01/gr_ref_joint: type fixed, parent robot_01/b3_link, child robot_01/gr_ref_link, origin xyz=0 -0.174 0 rpy=1.5708 0 -1.5708, axis 0 0 0
- added joint robot_01/m1_joint: type revolute, parent robot_01/base_link, child robot_01/m1_link, origin xyz=0.109379000000001 0.1082375 -0.0411999999999994 rpy=-1.5707963267949 0 0, axis 0 0 1, limit lower=0 upper=0 effort=0 velocity=0
- added joint robot_01/m1_r1_joint: type revolute, parent robot_01/m1_link, child robot_01/m1_r1_link, origin xyz=0.00228576835926038 -0.0386256329447082 0.0259400148238971 rpy=0.0417838903360263 -0.784524199152443 3.14159265358979, axis 0 0 -1, limit lower=0 upper=0 effort=0 velocity=0
- added joint robot_01/m1_r2_joint: type revolute, parent robot_01/m1_link, child robot_01/m1_r2_link, origin xyz=-0.0230770781232902 -0.0310582150591934 0.0259400148238969 rpy=-0.435348808486292 -0.676372195563374 3.14159265358979, axis 0 0 -1, limit lower=0 upper=0 effort=0 velocity=0
- added joint robot_01/m1_r3_joint: type revolute, parent robot_01/m1_link, child robot_01/m1_r3_link, origin xyz=-0.0376419032788015 -0.00895831317387084 0.0259400148238967 rpy=-0.758584186899929 -0.227513058576119 3.14159265358979, axis 0 0 -1, limit lower=0 upper=0 effort=0 velocity=0
- added joint robot_01/m1_r4_joint: type revolute, parent robot_01/m1_link, child robot_01/m1_r4_link, origin xyz=-0.0345936635470029 0.0173332830060698 0.0259400148238979 rpy=-0.68437497069708 0.421162065084444 3.14159265358979, axis 0 0 -1, limit lower=0 upper=0 effort=0 velocity=0
- added joint robot_01/m1_r5_joint: type revolute, parent robot_01/m1_link, child robot_01/m1_r5_link, origin xyz=-0.0153586641758173 0.0355144434294841 0.0259400148238974 rpy=-0.284497299709382 0.742588273963812 3.14159265358979, axis 0 0 -1, limit lower=0 upper=0 effort=0 velocity=0
- added joint robot_01/m1_r6_joint: type revolute, parent robot_01/m1_link, child robot_01/m1_r6_link, origin xyz=0.0110628248557701 0.0370780010731753 0.0259400148238963 rpy=0.203572981562908 0.764084510811395 3.14159265358979, axis 0 0 -1, limit lower=0 upper=0 effort=0 velocity=0
- added joint robot_01/m1_r7_joint: type revolute, parent robot_01/m1_link, child robot_01/m1_r7_link, origin xyz=0.0323078951877397 0.021292349938641 0.0259400148238976 rpy=0.631575557955456 0.503063157038392 3.14159265358979, axis 0 0 -1, limit lower=0 upper=0 effort=0 velocity=0
- added joint robot_01/m1_r8_joint: type revolute, parent robot_01/m1_link, child robot_01/m1_r8_link, origin xyz=0.0384357422991067 -0.00445622837028984 0.0259400148238975 rpy=0.778766107665016 -0.114663063476541 3.14159265358979, axis 0 0 -1, limit lower=0 upper=0 effort=0 velocity=0
- added joint robot_01/m1_r9_joint: type revolute, parent robot_01/m1_link, child robot_01/m1_r9_link, origin xyz=0.0265790784230276 -0.0281196878993006 0.0259400148238971 rpy=0.507192055712444 -0.628444159041816 3.14159265358979, axis 0 0 -1, limit lower=0 upper=0 effort=0 velocity=0
- added joint robot_01/m2_joint: type revolute, parent robot_01/base_link, child robot_01/m2_link, origin xyz=0.109379000000009 -0.1082375 -0.0412000000000078 rpy=1.5707963267949 0 0, axis 0 0 1, limit lower=0 upper=0 effort=0 velocity=0
- added joint robot_01/m2_r1_joint: type revolute, parent robot_01/m2_link, child robot_01/m2_r1_link, origin xyz=-0.00821200013368631 0.0378117350987201 0.0259400148239006 rpy=-0.150640941344919 0.773876910786465 0, axis 0 0 -1, limit lower=0 upper=0 effort=0 velocity=0
- added joint robot_01/m2_r2_joint: type revolute, parent robot_01/m2_link, child robot_01/m2_r2_link, origin xyz=-0.0305956718915099 0.0236868976203842 0.0259400148239005 rpy=-0.593332154467762 0.549321456352373 0, axis 0 0 -1, limit lower=0 upper=0 effort=0 velocity=0
- added joint robot_01/m2_r3_joint: type revolute, parent robot_01/m2_link, child robot_01/m2_r3_link, origin xyz=-0.0386632887382795 -0.00152130250507301 0.0259400148239004 rpy=-0.784625248127032 -0.0392968033136395 0, axis 0 0 -1, limit lower=0 upper=0 effort=0 velocity=0
- added joint robot_01/m2_r4_joint: type revolute, parent robot_01/m2_link, child robot_01/m2_r4_link, origin xyz=-0.0286399230898176 -0.0260176682810129 0.0259400148239003 rpy=-0.550819887589805 -0.591967673843851 0, axis 0 0 -1, limit lower=0 upper=0 effort=0 velocity=0
- added joint robot_01/m2_r5_joint: type revolute, parent robot_01/m2_link, child robot_01/m2_r5_link, origin xyz=-0.00521561913034017 -0.0383400779140923 0.0259400148239006 rpy=-0.0954587895624903 -0.780814086828851 0, axis 0 0 -1, limit lower=0 upper=0 effort=0 velocity=0
- added joint robot_01/m2_r6_joint: type revolute, parent robot_01/m2_link, child robot_01/m2_r6_link, origin xyz=0.0206491309853728 -0.0327227389886652 0.0259400148239008 rpy=0.386940296049201 -0.701990791531358 0, axis 0 0 -1, limit lower=0 upper=0 effort=0 velocity=0
- added joint robot_01/m2_r7_joint: type revolute, parent robot_01/m2_link, child robot_01/m2_r7_link, origin xyz=0.0368519232235012 -0.0117940668177069 0.0259400148239009 rpy=0.738876576610092 -0.295863549532841 0, axis 0 0 -1, limit lower=0 upper=0 effort=0 velocity=0
- added joint robot_01/m2_r8_joint: type revolute, parent robot_01/m2_link, child robot_01/m2_r8_link, origin xyz=0.0358112910218474 0.0146531802937085 0.0259400148239008 rpy=0.713442588606791 0.362011974105762 0, axis 0 0 -1, limit lower=0 upper=0 effort=0 velocity=0
- added joint robot_01/m2_r9_joint: type revolute, parent robot_01/m2_link, child robot_01/m2_r9_link, origin xyz=0.0180141577529039 0.0342440414937381 0.0259400148239017 rpy=0.335459767615501 0.724473747873283 0, axis 0 0 -1, limit lower=0 upper=0 effort=0 velocity=0
- added joint robot_01/m3_joint: type revolute, parent robot_01/base_link, child robot_01/m3_link, origin xyz=-0.109379000000082 0.1082375 -0.0411999999998636 rpy=-1.5707963267949 0 0, axis 0 0 1, limit lower=0 upper=0 effort=0 velocity=0
- added joint robot_01/m3_r1_joint: type revolute, parent robot_01/m3_link, child robot_01/m3_r1_link, origin xyz=0.00780265128511007 -0.0378983230538556 0.0259400148239009 rpy=-0.143078792692987 0.775020315169199 3.14159265358979, axis 0 0 -1, limit lower=0 upper=0 effort=0 velocity=0
- added joint robot_01/m3_r2_joint: type revolute, parent robot_01/m3_link, child robot_01/m3_r2_link, origin xyz=-0.0183833948283624 -0.034047247347707 0.0259400148239018 rpy=0.342614775914521 0.72161443573456 3.14159265358979, axis 0 0 -1, limit lower=0 upper=0 effort=0 velocity=0
- added joint robot_01/m3_r3_joint: type revolute, parent robot_01/m3_link, child robot_01/m3_r3_link, origin xyz=-0.0359676461929685 -0.0142650862145618 0.0259400148239008 rpy=0.717227786921772 0.353210967679924 3.14159265358979, axis 0 0 -1, limit lower=0 upper=0 effort=0 velocity=0
- added joint robot_01/m3_r4_joint: type revolute, parent robot_01/m3_link, child robot_01/m3_r4_link, origin xyz=-0.0367222361680236 0.0121918672971508 0.0259400148239009 rpy=0.735675192496111 -0.305243280167845 3.14159265358979, axis 0 0 -1, limit lower=0 upper=0 effort=0 velocity=0
- added joint robot_01/m3_r5_joint: type revolute, parent robot_01/m3_link, child robot_01/m3_r5_link, origin xyz=-0.0202940837178659 0.0329441106030149 0.025940014823901 rpy=0.379943833951376 -0.705316977204243 3.14159265358979, axis 0 0 -1, limit lower=0 upper=0 effort=0 velocity=0
- added joint robot_01/m3_r6_joint: type revolute, parent robot_01/m3_link, child robot_01/m3_r6_link, origin xyz=0.00562989604749835 0.0382814384247221 0.0259400148239009 rpy=-0.103067046354698 -0.780048810900469 3.14159265358979, axis 0 0 -1, limit lower=0 upper=0 effort=0 velocity=0
- added joint robot_01/m3_r7_joint: type revolute, parent robot_01/m3_link, child robot_01/m3_r7_link, origin xyz=0.0289195848829134 0.0257064557567044 0.0259400148239008 rpy=-0.556828855344444 -0.586408226610345 3.14159265358979, axis 0 0 -1, limit lower=0 upper=0 effort=0 velocity=0
- added joint robot_01/m3_r8_joint: type revolute, parent robot_01/m3_link, child robot_01/m3_r8_link, origin xyz=0.0386774785462282 0.00110313674469228 0.0259400148239009 rpy=-0.784991758153164 -0.0285021092700616 3.14159265358979, axis 0 0 -1, limit lower=0 upper=0 effort=0 velocity=0
- added joint robot_01/m3_r9_joint: type revolute, parent robot_01/m3_link, child robot_01/m3_r9_link, origin xyz=0.0303377501454697 -0.0240163522101604 0.0259400148239009 rpy=-0.587657847652812 0.555491477512066 3.14159265358979, axis 0 0 -1, limit lower=0 upper=0 effort=0 velocity=0
- added joint robot_01/m4_joint: type revolute, parent robot_01/base_link, child robot_01/m4_link, origin xyz=-0.109379 -0.1082375 -0.0412000000000007 rpy=1.5707963267949 0 0, axis 0 0 1, limit lower=0 upper=0 effort=0 velocity=0
- added joint robot_01/m4_r1_joint: type revolute, parent robot_01/m4_link, child robot_01/m4_r1_link, origin xyz=0.0131833857778636 0.036378051030856 0.025940014823897 rpy=-0.243316166077614 -0.754568490942695 0, axis 0 0 -1, limit lower=0 upper=0 effort=0 velocity=0
- added joint robot_01/m4_r2_joint: type revolute, parent robot_01/m4_link, child robot_01/m4_r2_link, origin xyz=-0.0132843010505526 0.0363413208754141 0.0259400148238971 rpy=0.245216782606616 -0.754064372015612 0, axis 0 0 1, limit lower=0 upper=0 effort=0 velocity=0
- added joint robot_01/m4_r3_joint: type revolute, parent robot_01/m4_link, child robot_01/m4_r3_link, origin xyz=-0.0335361157788547 0.0193000827935733 0.025940014823897 rpy=0.659678052589828 -0.46268531073941 0, axis 0 0 -1, limit lower=0 upper=0 effort=0 velocity=0
- added joint robot_01/m4_r4_joint: type revolute, parent robot_01/m4_link, child robot_01/m4_r4_link, origin xyz=-0.0380960092218195 -0.0067718785239083 0.0259400148238974 rpy=0.770080701636149 0.173259892811608 0, axis 0 0 -1, limit lower=0 upper=0 effort=0 velocity=0
- added joint robot_01/m4_r5_joint: type revolute, parent robot_01/m4_link, child robot_01/m4_r5_link, origin xyz=-0.0248303565599136 -0.0296752026190064 0.0259400148238976 rpy=0.470988454485595 0.654252157673773 0, axis 0 0 -1, limit lower=0 upper=0 effort=0 velocity=0
- added joint robot_01/m4_r6_joint: type revolute, parent robot_01/m4_link, child robot_01/m4_r6_link, origin xyz=5.36958950512478E-05 -0.0386931696055349 0.0259400148238963 rpy=-0.000981276577522423 0.785397681945272 0, axis 0 0 -1, limit lower=0 upper=0 effort=0 velocity=0
- added joint robot_01/m4_r7_joint: type revolute, parent robot_01/m4_link, child robot_01/m4_r7_link, origin xyz=0.0249126234439565 -0.0296061725069484 0.0259400148238975 rpy=-0.472676273649131 0.653127875272481 0, axis 0 0 -1, limit lower=0 upper=0 effort=0 velocity=0
- added joint robot_01/m4_r8_joint: type revolute, parent robot_01/m4_link, child robot_01/m4_r8_link, origin xyz=0.0381146576104692 -0.0066661182564095 0.0259400148238981 rpy=-0.770555550274693 0.170606597523424 0, axis 0 0 -1, limit lower=0 upper=0 effort=0 velocity=0
- added joint robot_01/m4_r9_joint: type revolute, parent robot_01/m4_link, child robot_01/m4_r9_link, origin xyz=0.0334824198838078 0.019393086811959 0.025940014823897 rpy=-0.658436825683223 -0.464608212552487 0, axis 0 0 -1, limit lower=0 upper=0 effort=0 velocity=0
- added joint robot_01/marker_joint: type prismatic, parent robot_01/base_link, child marker_id_01, origin xyz=-0.0874999999999998 0 0.000999999999999876 rpy=0 0 0, axis 0 0 1, limit lower=0 upper=0 effort=0 velocity=0
- added joint robot_01/p1_joint: type revolute, parent robot_01/b3_link, child robot_01/p1_link, origin xyz=0 -0.099605 0.0135 rpy=1.5708 0 -1.5708, axis 0 0 -1, limit lower=0 upper=0 effort=0 velocity=0, mimic joint=robot_01/p2_joint multiplier=-1 offset=0
- added joint robot_01/p2_joint: type revolute, parent robot_01/b3_link, child robot_01/p2_link, origin xyz=0 -0.099605 -0.0135 rpy=1.5708 0 -1.5708, axis 0 0 1, limit lower=0 upper=0 effort=0 velocity=0, mimic joint=robot_01/p1_joint multiplier=-1 offset=0
