Commit message: Both robots working on rviz2

File: src/robot_custom_description/models/robot_01/model.urdf (robot description, URDF)
Before this commit: robot robot_01, 48 links, 47 joints
Links:
- link robot_01/b3_link: mass 0.194452851189113 -> 0.194452851189114
- link robot_01/base_link: mass 1.30966382009507 -> 1.3097
- link robot_01/gr_ref_link: mass 0.0005 -> 0.000500000000000001
- link robot_01/m1_link: mass 0.348747920870875 -> 0.34875
- link robot_01/m3_r5_link: mass 0.00929201442640375 -> 0.00929201442640374
- link robot_01/p1_link: mass 0.0032658 -> 0.00326579291252288
- link robot_01/p2_link: mass 0.0032658 -> 0.00326579291252288
Joints:
- removed joint robot_01/marker_joint
- added joint robot_01/base_joint: type fixed, parent marker_id_01, child robot_01/base_link, origin xyz=0.0875 0 -0.001 rpy=0 0 0, axis 0 0 0
- joint robot_01/b1_joint: origin xyz=0.0749999999999994 0 0.0620000000000007 rpy=-1.5707963267949 0 0 -> xyz=0.075 0 0.062 rpy=-1.5708 0 0
- joint robot_01/b3_joint: origin xyz=0 -0.0699999999999995 0 rpy=0 0 0 -> xyz=0 -0.07 0 rpy=0 0 0
- joint robot_01/m1_joint: origin xyz=0.109379000000001 0.1082375 -0.0411999999999994 rpy=-1.5707963267949 0 0 -> xyz=0.10938 0.10824 -0.0412 rpy=-1.5708 0 0
- joint robot_01/m1_r1_joint: origin xyz=0.00228576835926038 -0.0386256329447082 0.0259400148238971 rpy=0.0417838903360263 -0.784524199152443 3.14159265358979 -> xyz=0.0022858 -0.038626 0.02594 rpy=0.041784 -0.78452 3.1416
- joint robot_01/m2_joint: origin xyz=0.109379000000009 -0.1082375 -0.0412000000000078 rpy=1.5707963267949 0 0 -> xyz=0.10938 -0.10824 -0.0412 rpy=1.5708 0 0
- joint robot_01/m3_joint: origin xyz=-0.109379000000082 0.1082375 -0.0411999999998636 rpy=-1.5707963267949 0 0 -> xyz=-0.10938 0.10824 -0.0412 rpy=-1.5708 0 0
- joint robot_01/m4_joint: origin xyz=-0.109379 -0.1082375 -0.0412000000000007 rpy=1.5707963267949 0 0 -> xyz=-0.10938 -0.10824 -0.0412 rpy=1.5708 0 0
- joint robot_01/p2_joint: mimic joint=robot_01/p1_joint multiplier=-1 offset=0 -> (none)
