Commit message: Update measure arm

File: src/robot_custom_description/models/robot_01/model.urdf (robot description, URDF)
Before this commit: robot robot_01, 49 links, 48 joints
Links:
- link robot_01/b1_link: mass 0.233473387976464 -> 0.233473387976465
- link robot_01/base_arm: mass 0.19395 -> 0.193946324100217
- link robot_01/m2_r3_link: mass 0.00929201442640374 -> 0.00929201442640375
- link robot_01/m3_r5_link: mass 0.00929201442640374 -> 0.00929201442640375
Joints:
- joint robot_01/base_joint: origin xyz=0.0875 0 -0.001 rpy=0 0 0 -> xyz=0.0874999999999998 0 -0.000999999999999876 rpy=0 0 0
- joint robot_01/m1_joint: origin xyz=0.10938 0.10824 -0.0412 rpy=-1.5708 0 0 -> xyz=0.109379000000001 0.1082375 -0.0411999999999994 rpy=-1.5707963267949 0 0
- joint robot_01/m3_r3_joint: origin xyz=-0.0183833948283624 -0.034047247347707 0.0259400148239018 rpy=0.342614775914521 0.72161443573456 3.14159265358979 -> xyz=-0.035968 -0.014265 0.02594 rpy=0.71723 0.35321 3.1416
- joint robot_01/m3_r4_joint: origin xyz=-0.0367222361680236 0.0121918672971508 0.0259400148239009 rpy=0.735675192496111 -0.305243280167845 3.14159265358979 -> xyz=-0.036722 0.012192 0.02594 rpy=0.73568 -0.30524 3.1416
- joint robot_01/m4_r9_joint: origin xyz=0.033482 0.019393 0.02594 rpy=-0.65844 -0.46461 0 -> xyz=0.0334824198838078 0.019393086811959 0.025940014823897 rpy=-0.658436825683223 -0.464608212552487 0
- joint robot_01/p2_joint: origin xyz=0.099605 0 0.0135 rpy=-1.5708 0 0 -> xyz=0.0996053139252814 0 0.0135000000000004 rpy=-1.5707963267949 0 0

File: src/robot_custom_description/models/robot_01/model_backup.urdf (robot description, URDF)
Before this commit: robot robot_01, 48 links, 47 joints
Links:
- added link robot_01/base_arm, mass 0.19395; collision mesh filename=package://robot_custom_description/models/robot_01/meshes/r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; visual mesh filename=package://robot_custom_description/models/robot_01/meshes/r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
- link robot_01/b1_link: geometry collision mesh filename=package://robot_custom_description/models/robot_01/meshes/r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; visual mesh filename=package://robot_custom_description/models/robot_01/meshes/r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
- link robot_01/b2_link: geometry collision mesh filename=package://robot_custom_description/models/robot_01/meshes/r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; visual mesh filename=package://robot_custom_description/models/robot_01/meshes/r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
- link robot_01/b3_link: geometry collision mesh filename=package://robot_custom_description/models/robot_01/meshes/r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; visual mesh filename=package://robot_custom_description/models/robot_01/meshes/r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
- link robot_01/base_link: mass 1.3097 -> 1.11571749599485; geometry collision mesh filename=package://robot_custom_description/models/robot_01/meshes/r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; visual mesh filename=package://robot_custom_description/models/robot_01/meshes/r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
- link robot_01/gr_ref_link: geometry collision mesh filename=package://robot_custom_description/models/robot_01/meshes/r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; visual mesh filename=package://robot_custom_description/models/robot_01/meshes/r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
- link robot_01/m1_link: mass 0.34875 -> 0.348747920870875; geometry collision mesh filename=package://robot_custom_description/models/robot_01/meshes/r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; visual mesh filename=package://robot_custom_description/models/robot_01/meshes/r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
- link robot_01/m1_r1_link: geometry collision mesh filename=package://robot_custom_description/models/robot_01/meshes/r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; visual mesh filename=package://robot_custom_description/models/robot_01/meshes/r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
- link robot_01/m1_r2_link: geometry collision mesh filename=package://robot_custom_description/models/robot_01/meshes/r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; visual mesh filename=package://robot_custom_description/models/robot_01/meshes/r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
- link robot_01/m1_r3_link: geometry collision mesh filename=package://robot_custom_description/models/robot_01/meshes/r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; visual mesh filename=package://robot_custom_description/models/robot_01/meshes/r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
- link robot_01/m1_r4_link: geometry collision mesh filename=package://robot_custom_description/models/robot_01/meshes/r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; visual mesh filename=package://robot_custom_description/models/robot_01/meshes/r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
- link robot_01/m1_r5_link: geometry collision mesh filename=package://robot_custom_description/models/robot_01/meshes/r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; visual mesh filename=package://robot_custom_description/models/robot_01/meshes/r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
- link robot_01/m1_r6_link: geometry collision mesh filename=package://robot_custom_description/models/robot_01/meshes/r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; visual mesh filename=package://robot_custom_description/models/robot_01/meshes/r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
- link robot_01/m1_r7_link: geometry collision mesh filename=package://robot_custom_description/models/robot_01/meshes/r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; visual mesh filename=package://robot_custom_description/models/robot_01/meshes/r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
- link robot_01/m1_r8_link: geometry collision mesh filename=package://robot_custom_description/models/robot_01/meshes/r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; visual mesh filename=package://robot_custom_description/models/robot_01/meshes/r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
- link robot_01/m1_r9_link: geometry collision mesh filename=package://robot_custom_description/models/robot_01/meshes/r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; visual mesh filename=package://robot_custom_description/models/robot_01/meshes/r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
- link robot_01/m2_link: geometry collision mesh filename=package://robot_custom_description/models/robot_01/meshes/r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; visual mesh filename=package://robot_custom_description/models/robot_01/meshes/r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
- link robot_01/m2_r1_link: geometry collision mesh filename=package://robot_custom_description/models/robot_01/meshes/r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; visual mesh filename=package://robot_custom_description/models/robot_01/meshes/r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
- link robot_01/m2_r2_link: geometry collision mesh filename=package://robot_custom_description/models/robot_01/meshes/r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; visual mesh filename=package://robot_custom_description/models/robot_01/meshes/r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
- link robot_01/m2_r3_link: geometry collision mesh filename=package://robot_custom_description/models/robot_01/meshes/r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; visual mesh filename=package://robot_custom_description/models/robot_01/meshes/r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
- link robot_01/m2_r4_link: geometry collision mesh filename=package://robot_custom_description/models/robot_01/meshes/r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; visual mesh filename=package://robot_custom_description/models/robot_01/meshes/r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
- link robot_01/m2_r5_link: geometry collision mesh filename=package://robot_custom_description/models/robot_01/meshes/r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; visual mesh filename=package://robot_custom_description/models/robot_01/meshes/r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
- link robot_01/m2_r6_link: geometry collision mesh filename=package://robot_custom_description/models/robot_01/meshes/r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; visual mesh filename=package://robot_custom_description/models/robot_01/meshes/r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
- link robot_01/m2_r7_link: geometry collision mesh filename=package://robot_custom_description/models/robot_01/meshes/r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; visual mesh filename=package://robot_custom_description/models/robot_01/meshes/r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
- link robot_01/m2_r8_link: geometry collision mesh filename=package://robot_custom_description/models/robot_01/meshes/r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; visual mesh filename=package://robot_custom_description/models/robot_01/meshes/r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
- link robot_01/m2_r9_link: geometry collision mesh filename=package://robot_custom_description/models/robot_01/meshes/r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; visual mesh filename=package://robot_custom_description/models/robot_01/meshes/r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
- link robot_01/m3_link: geometry collision mesh filename=package://robot_custom_description/models/robot_01/meshes/r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; visual mesh filename=package://robot_custom_description/models/robot_01/meshes/r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
- link robot_01/m3_r1_link: geometry collision mesh filename=package://robot_custom_description/models/robot_01/meshes/r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; visual mesh filename=package://robot_custom_description/models/robot_01/meshes/r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
- link robot_01/m3_r2_link: geometry collision mesh filename=package://robot_custom_description/models/robot_01/meshes/r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; visual mesh filename=package://robot_custom_description/models/robot_01/meshes/r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
- link robot_01/m3_r3_link: geometry collision mesh filename=package://robot_custom_description/models/robot_01/meshes/r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; visual mesh filename=package://robot_custom_description/models/robot_01/meshes/r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
- link robot_01/m3_r4_link: geometry collision mesh filename=package://robot_custom_description/models/robot_01/meshes/r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; visual mesh filename=package://robot_custom_description/models/robot_01/meshes/r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
- link robot_01/m3_r5_link: geometry collision mesh filename=package://robot_custom_description/models/robot_01/meshes/r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; visual mesh filename=package://robot_custom_description/models/robot_01/meshes/r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
- link robot_01/m3_r6_link: geometry collision mesh filename=package://robot_custom_description/models/robot_01/meshes/r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; visual mesh filename=package://robot_custom_description/models/robot_01/meshes/r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
- link robot_01/m3_r7_link: geometry collision mesh filename=package://robot_custom_description/models/robot_01/meshes/r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; visual mesh filename=package://robot_custom_description/models/robot_01/meshes/r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
- link robot_01/m3_r8_link: geometry collision mesh filename=package://robot_custom_description/models/robot_01/meshes/r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; visual mesh filename=package://robot_custom_description/models/robot_01/meshes/r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
- link robot_01/m3_r9_link: geometry collision mesh filename=package://robot_custom_description/models/robot_01/meshes/r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; visual mesh filename=package://robot_custom_description/models/robot_01/meshes/r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
- link robot_01/m4_link: geometry collision mesh filename=package://robot_custom_description/models/robot_01/meshes/r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; visual mesh filename=package://robot_custom_description/models/robot_01/meshes/r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
- link robot_01/m4_r1_link: geometry collision mesh filename=package://robot_custom_description/models/robot_01/meshes/r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; visual mesh filename=package://robot_custom_description/models/robot_01/meshes/r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
- link robot_01/m4_r2_link: geometry collision mesh filename=package://robot_custom_description/models/robot_01/meshes/r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; visual mesh filename=package://robot_custom_description/models/robot_01/meshes/r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
- link robot_01/m4_r3_link: geometry collision mesh filename=package://robot_custom_description/models/robot_01/meshes/r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; visual mesh filename=package://robot_custom_description/models/robot_01/meshes/r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
- link robot_01/m4_r4_link: geometry collision mesh filename=package://robot_custom_description/models/robot_01/meshes/r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; visual mesh filename=package://robot_custom_description/models/robot_01/meshes/r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
- link robot_01/m4_r5_link: geometry collision mesh filename=package://robot_custom_description/models/robot_01/meshes/r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; visual mesh filename=package://robot_custom_description/models/robot_01/meshes/r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
- link robot_01/m4_r6_link: geometry collision mesh filename=package://robot_custom_description/models/robot_01/meshes/r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; visual mesh filename=package://robot_custom_description/models/robot_01/meshes/r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
- link robot_01/m4_r7_link: geometry collision mesh filename=package://robot_custom_description/models/robot_01/meshes/r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; visual mesh filename=package://robot_custom_description/models/robot_01/meshes/r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
- link robot_01/m4_r8_link: geometry collision mesh filename=package://robot_custom_description/models/robot_01/meshes/r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; visual mesh filename=package://robot_custom_description/models/robot_01/meshes/r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
- link robot_01/m4_r9_link: geometry collision mesh filename=package://robot_custom_description/models/robot_01/meshes/r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; visual mesh filename=package://robot_custom_description/models/robot_01/meshes/r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
- link robot_01/p1_link: geometry collision mesh filename=package://robot_custom_description/models/robot_01/meshes/r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; visual mesh filename=package://robot_custom_description/models/robot_01/meshes/r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
- link robot_01/p2_link: geometry collision mesh filename=package://robot_custom_description/models/robot_01/meshes/r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; visual mesh filename=package://robot_custom_description/models/robot_01/meshes/r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
Joints:
- added joint robot_01/base_arm_joint: type fixed, parent robot_01/base_link, child robot_01/base_arm, origin xyz=0.075 0 0.062 rpy=1.5708 -1.5708 0, axis 0 0 0
- joint robot_01/b1_joint: axis 0 0 1 -> 0 0 -1; limit lower=0 upper=0 effort=0 velocity=0 -> lower=-1.5 upper=1.5 effort=-1 velocity=1.5; origin xyz=0.075 0 0.062 rpy=-1.5708 0 0 -> xyz=0 0 0 rpy=0 0 0; parent robot_01/base_link -> robot_01/base_arm
- joint robot_01/b2_joint: axis 0 0 1 -> 0 0 -1; limit lower=0 upper=0 effort=0 velocity=0 -> lower=-1.5 upper=1.5 effort=-1 velocity=1.5; origin xyz=0 -0.075 0 rpy=0 0 0 -> xyz=0.075 0 0 rpy=0 0 0
- joint robot_01/b3_joint: axis 0 0 1 -> 0 0 -1; limit lower=0 upper=0 effort=0 velocity=0 -> lower=-1.5 upper=1.5 effort=-1 velocity=1.5; origin xyz=0 -0.07 0 rpy=0 0 0 -> xyz=0.0699999999999995 0 0 rpy=0 0 0
- joint robot_01/gr_ref_joint: origin xyz=0 -0.174 0 rpy=1.5708 0 -1.5708 -> xyz=0.174 0 0 rpy=-1.5707963267949 0 0
- joint robot_01/m1_joint: limit lower=0 upper=0 effort=0 velocity=0 -> lower=-1E+50 upper=1E+50 effort=-1 velocity=-1
- joint robot_01/m1_r1_joint: limit lower=0 upper=0 effort=0 velocity=0 -> lower=-1E+50 upper=1E+50 effort=-1 velocity=-1; origin xyz=0.0022858 -0.038626 0.02594 rpy=0.041784 -0.78452 3.1416 -> xyz=0.00228576835926038 -0.0386256329447082 0.0259400148238971 rpy=0.0417838903360263 -0.784524199152443 3.14159265358979
- joint robot_01/m1_r2_joint: limit lower=0 upper=0 effort=0 velocity=0 -> lower=-1E+50 upper=1E+50 effort=-1 velocity=-1
- joint robot_01/m1_r3_joint: limit lower=0 upper=0 effort=0 velocity=0 -> lower=-1E+50 upper=1E+50 effort=-1 velocity=-1
- joint robot_01/m1_r4_joint: limit lower=0 upper=0 effort=0 velocity=0 -> lower=-1E+50 upper=1E+50 effort=-1 velocity=-1
- joint robot_01/m1_r5_joint: limit lower=0 upper=0 effort=0 velocity=0 -> lower=-1E+50 upper=1E+50 effort=-1 velocity=-1
- joint robot_01/m1_r6_joint: limit lower=0 upper=0 effort=0 velocity=0 -> lower=-1E+50 upper=1E+50 effort=-1 velocity=-1
- joint robot_01/m1_r7_joint: limit lower=0 upper=0 effort=0 velocity=0 -> lower=-1E+50 upper=1E+50 effort=-1 velocity=-1
- joint robot_01/m1_r8_joint: limit lower=0 upper=0 effort=0 velocity=0 -> lower=-1E+50 upper=1E+50 effort=-1 velocity=-1
- joint robot_01/m1_r9_joint: limit lower=0 upper=0 effort=0 velocity=0 -> lower=-1E+50 upper=1E+50 effort=-1 velocity=-1
- joint robot_01/m2_joint: limit lower=0 upper=0 effort=0 velocity=0 -> lower=-1E+50 upper=1E+50 effort=-1 velocity=-1; origin xyz=0.10938 -0.10824 -0.0412 rpy=1.5708 0 0 -> xyz=0.109379000000009 -0.1082375 -0.0412000000000078 rpy=1.5707963267949 0 0
- joint robot_01/m2_r1_joint: limit lower=0 upper=0 effort=0 velocity=0 -> lower=-1E+50 upper=1E+50 effort=-1 velocity=-1
- joint robot_01/m2_r2_joint: limit lower=0 upper=0 effort=0 velocity=0 -> lower=-1E+50 upper=1E+50 effort=-1 velocity=-1
- joint robot_01/m2_r3_joint: limit lower=0 upper=0 effort=0 velocity=0 -> lower=-1E+50 upper=1E+50 effort=-1 velocity=-1
- joint robot_01/m2_r4_joint: limit lower=0 upper=0 effort=0 velocity=0 -> lower=-1E+50 upper=1E+50 effort=-1 velocity=-1
- joint robot_01/m2_r5_joint: limit lower=0 upper=0 effort=0 velocity=0 -> lower=-1E+50 upper=1E+50 effort=-1 velocity=-1
- joint robot_01/m2_r6_joint: limit lower=0 upper=0 effort=0 velocity=0 -> lower=-1E+50 upper=1E+50 effort=-1 velocity=-1
- joint robot_01/m2_r7_joint: limit lower=0 upper=0 effort=0 velocity=0 -> lower=-1E+50 upper=1E+50 effort=-1 velocity=-1
- joint robot_01/m2_r8_joint: limit lower=0 upper=0 effort=0 velocity=0 -> lower=-1E+50 upper=1E+50 effort=-1 velocity=-1
- joint robot_01/m2_r9_joint: limit lower=0 upper=0 effort=0 velocity=0 -> lower=-1E+50 upper=1E+50 effort=-1 velocity=-1
- joint robot_01/m3_joint: limit lower=0 upper=0 effort=0 velocity=0 -> lower=-1E+50 upper=1E+50 effort=-1 velocity=-1; origin xyz=-0.10938 0.10824 -0.0412 rpy=-1.5708 0 0 -> xyz=-0.109379000000082 0.1082375 -0.0411999999998636 rpy=-1.5707963267949 0 0
- joint robot_01/m3_r1_joint: limit lower=0 upper=0 effort=0 velocity=0 -> lower=-1E+50 upper=1E+50 effort=-1 velocity=-1
- joint robot_01/m3_r2_joint: limit lower=0 upper=0 effort=0 velocity=0 -> lower=-1E+50 upper=1E+50 effort=-1 velocity=-1
- joint robot_01/m3_r3_joint: limit lower=0 upper=0 effort=0 velocity=0 -> lower=-1E+50 upper=1E+50 effort=-1 velocity=-1; origin xyz=-0.0359676461929685 -0.0142650862145618 0.0259400148239008 rpy=0.717227786921772 0.353210967679924 3.14159265358979 -> xyz=-0.0183833948283624 -0.034047247347707 0.0259400148239018 rpy=0.342614775914521 0.72161443573456 3.14159265358979
- joint robot_01/m3_r4_joint: limit lower=0 upper=0 effort=0 velocity=0 -> lower=-1E+50 upper=1E+50 effort=-1 velocity=-1
- joint robot_01/m3_r5_joint: limit lower=0 upper=0 effort=0 velocity=0 -> lower=-1E+50 upper=1E+50 effort=-1 velocity=-1
- joint robot_01/m3_r6_joint: limit lower=0 upper=0 effort=0 velocity=0 -> lower=-1E+50 upper=1E+50 effort=-1 velocity=-1
- joint robot_01/m3_r7_joint: limit lower=0 upper=0 effort=0 velocity=0 -> lower=-1E+50 upper=1E+50 effort=-1 velocity=-1
- joint robot_01/m3_r8_joint: limit lower=0 upper=0 effort=0 velocity=0 -> lower=-1E+50 upper=1E+50 effort=-1 velocity=-1
- joint robot_01/m3_r9_joint: limit lower=0 upper=0 effort=0 velocity=0 -> lower=-1E+50 upper=1E+50 effort=-1 velocity=-1
- joint robot_01/m4_joint: limit lower=0 upper=0 effort=0 velocity=0 -> lower=-1E+50 upper=1E+50 effort=-1 velocity=-1; origin xyz=-0.10938 -0.10824 -0.0412 rpy=1.5708 0 0 -> xyz=-0.109379 -0.1082375 -0.0412000000000007 rpy=1.5707963267949 0 0
- joint robot_01/m4_r1_joint: limit lower=0 upper=0 effort=0 velocity=0 -> lower=-1E+50 upper=1E+50 effort=-1 velocity=-1
- joint robot_01/m4_r2_joint: limit lower=0 upper=0 effort=0 velocity=0 -> lower=-1E+50 upper=1E+50 effort=-1 velocity=-1
- joint robot_01/m4_r3_joint: limit lower=0 upper=0 effort=0 velocity=0 -> lower=-1E+50 upper=1E+50 effort=-1 velocity=-1
- joint robot_01/m4_r4_joint: limit lower=0 upper=0 effort=0 velocity=0 -> lower=-1E+50 upper=1E+50 effort=-1 velocity=-1
- joint robot_01/m4_r5_joint: limit lower=0 upper=0 effort=0 velocity=0 -> lower=-1E+50 upper=1E+50 effort=-1 velocity=-1
- joint robot_01/m4_r6_joint: limit lower=0 upper=0 effort=0 velocity=0 -> lower=-1E+50 upper=1E+50 effort=-1 velocity=-1
- joint robot_01/m4_r7_joint: limit lower=0 upper=0 effort=0 velocity=0 -> lower=-1E+50 upper=1E+50 effort=-1 velocity=-1
- joint robot_01/m4_r8_joint: limit lower=0 upper=0 effort=0 velocity=0 -> lower=-1E+50 upper=1E+50 effort=-1 velocity=-1
- joint robot_01/m4_r9_joint: limit lower=0 upper=0 effort=0 velocity=0 -> lower=-1E+50 upper=1E+50 effort=-1 velocity=-1; origin xyz=0.0334824198838078 0.019393086811959 0.025940014823897 rpy=-0.658436825683223 -0.464608212552487 0 -> xyz=0.033482 0.019393 0.02594 rpy=-0.65844 -0.46461 0
- joint robot_01/p1_joint: limit lower=0 upper=0 effort=0 velocity=0 -> lower=-1 upper=1 effort=-1 velocity=1; mimic joint=robot_01/p2_joint multiplier=-1 offset=0 -> (none); origin xyz=0 -0.099605 0.0135 rpy=1.5708 0 -1.5708 -> xyz=0.099605 0 -0.0135 rpy=-1.5708 0 0
- joint robot_01/p2_joint: limit lower=0 upper=0 effort=0 velocity=0 -> lower=-1 upper=1 effort=-1 velocity=1; origin xyz=0 -0.099605 -0.0135 rpy=1.5708 0 -1.5708 -> xyz=0.099605 0 0.0135 rpy=-1.5708 0 0
