Commit message: Update

File: src/robot_custom_description/models/cube_id_11/model.urdf (robot description, URDF)
Before this commit: robot single_cube_02, 2 links, 1 joints
Links:
- removed link marker_id_12
- removed link single_cube_02/cube_link
- added link cube_id_11/cube_link, mass 0.2; collision mesh filename=package://robot_custom_description/models/cube_id_11/meshes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; visual mesh filename=package://robot_custom_description/models/cube_id_11/meshes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
- added link marker_id_11, mass 0.0144; visual mesh filename=package://robot_custom_description/models/markers/marker_11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
Joints:
- removed joint single_cube_02/cube_joint
- added joint cube_id_11/cube_joint: type fixed, parent marker_id_11, child cube_id_11/cube_link, origin xyz=0 0 -0.051 rpy=0 0 0, axis 0 0 0

File: src/robot_custom_description/models/cube_id_12/model.urdf (robot description, URDF)
Before this commit: robot single_cube_01, 2 links, 1 joints
Links:
- removed link marker_id_11
- removed link single_cube_01/cube_link
- added link cube_id_12/cube_link, mass 0.2; collision mesh filename=package://robot_custom_description/models/cube_id_12/meshes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; visual mesh filename=package://robot_custom_description/models/cube_id_12/meshes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
- added link marker_id_12, mass 0.0144; visual mesh filename=package://robot_custom_description/models/markers/marker_12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
Joints:
- removed joint single_cube_01/cube_joint
- added joint cube_id_12/cube_joint: type fixed, parent marker_id_12, child cube_id_12/cube_link, origin xyz=0 0 -0.051 rpy=0 0 0, axis 0 0 0

File: src/robot_custom_description/models/cube_id_21/model.urdf (robot description, URDF)
Before this commit: robot double_cube_01, 2 links, 1 joints
Links:
- removed link double_cube_01/cube_link
- added link cube_id_21/cube_link, mass 0.5; collision mesh filename=package://robot_custom_description/models/cube_id_21/meshes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; visual mesh filename=package://robot_custom_description/models/cube_id_21/meshes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
Joints:
- removed joint double_cube_01/cube_joint
- added joint cube_id_21/cube_joint: type fixed, parent marker_id_21, child cube_id_21/cube_link, origin xyz=0 0 -0.051 rpy=0 0 0, axis 0 0 0

Commit message: Update models

File: src/robot_custom_description/models/cube_id_11/model.urdf (robot description, URDF)
Before this commit: robot cube_id_11, 2 links, 1 joints
Links:
- link cube_id_11/cube_link: mass 0.2 -> 0.02
Joints:
- joint cube_id_11/cube_joint: origin xyz=0 0 -0.051 rpy=0 0 0 -> xyz=0 0 -0.076 rpy=0 0 0

File: src/robot_custom_description/models/cube_id_11/model_old.urdf (robot description, URDF)
Before this commit: robot cube_id_21, 2 links, 1 joints
Links:
- removed link cube_id_21/cube_link
- removed link marker_id_21
- added link cube_id_11/cube_link, mass 0.2; collision mesh filename=package://robot_custom_description/models/cube_id_11/meshes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; visual mesh filename=package://robot_custom_description/models/cube_id_11/meshes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
- added link marker_id_11, mass 0.0144; visual mesh filename=package://robot_custom_description/models/markers/marker_11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
Joints:
- removed joint cube_id_21/cube_joint
- added joint cube_id_11/cube_joint: type fixed, parent marker_id_11, child cube_id_11/cube_link, origin xyz=0 0 -0.051 rpy=0 0 0, axis 0 0 0

File: src/robot_custom_description/models/cube_id_12/model.urdf (robot description, URDF)
Before this commit: robot cube_id_12, 2 links, 1 joints
Links:
- link cube_id_12/cube_link: mass 0.2 -> 0.02
Joints:
- joint cube_id_12/cube_joint: origin xyz=0 0 -0.051 rpy=0 0 0 -> xyz=0 0 -0.076 rpy=0 0 0
